File: schematics/main_board/_autosave-main_board.sch (KiCad schematic (older format))
At the start: 56 parts, among them J1 USB_B_Micro, M1 Motor_DC, M2 Motor_DC, M3 Motor_DC, M4 Motor_DC, Q1 BC817, Q2 2N7002, Q3 2N7002, Q4 2N7002, Q5 2N7002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

Commit message: Changed some footprints, added some traces
Parts:
- D1: footprint Diode_SMD:D_SOT-23_ANK -> Package_TO_SOT_SMD:SOT-23
Connections:
- net M1 is gone; now on net S1: U1.17 (PA3)
- net M4 is gone; now on net S4: U1.16 (PA2)
- net VBAT_PAD is gone; now on net BAT+: BT1.1 (+), D4.1 (K), D5.1 (K), D6.1 (K), D7.1 (K), M1.1 (+), M2.1 (+), M3.1 (+), M4.1 (+), U1.9 (PC1)
- net 5V_EXTERNAL renamed BAT+
Changed lines of the file:
@@
 	10300 1900 10500 1900
 Text GLabel 10400 2100 2    50   Output ~ 0
-M4
+S4
 Text GLabel 10400 2200 2    50   Output ~ 0
-M1
+S1
 $Comp
 L Sensor_Motion:MPU-6000 U3
@@
 	8300 3100 8300 3400
 Text GLabel 8800 3700 0    50   Output ~ 0
-VBAT_PAD
+BAT+
 Text GLabel 8800 3800 0    50   Output ~ 0
 RSSI_PAD
@@
 F 0 "D1" V 1554 4738 50  0000 L CNN
 F 1 "BAT54C" V 1645 4738 50  0000 L CNN
-F 2 "Diode_SMD:D_SOT-23_ANK" H 1675 4775 50  0001 L CNN
+F 2 "Package_TO_SOT_SMD:SOT-23" H 1675 4775 50  0001 L CNN
 F 3 "http://www.diodes.com/_files/datasheets/ds11005.pdf" H 1520 4650 50  0001 C CNN
 	1    1600 4650
@@
 5V_USB
 Text GLabel 1550 5050 0    50   Input ~ 0
-5V_EXTERNAL
+BAT+
 Wire Wire Line
 	1550 4250 1600 4250
@@
 $EndComp
 Text GLabel 2050 6000 0    50   Input ~ 0
-5V_EXTERNAL
+BAT+
 Text GLabel 2300 6550 2    50   Output ~ 0
 UART1_RX
@@
 $EndComp
 Text GLabel 3800 4250 2    50   Output ~ 0
-VBAT_PAD
+BAT+
 Wire Wire Line
 	3650 4450 3650 4250
@@
 	3650 4850 3650 4750
 Text GLabel 5500 6550 1    50   Output ~ 0
-VBAT_PAD
+BAT+
 $Comp
 L Device:R R9
@@
 $EndComp
 Text GLabel 7600 6600 1    50   Output ~ 0
-VBAT_PAD
+BAT+
 $Comp
 L Device:R R13
@@
 $EndComp
 Text GLabel 5500 9000 1    50   Output ~ 0
-VBAT_PAD
+BAT+
 $Comp
 L Device:R R10
@@
 $EndComp
 Text GLabel 7600 9050 1    50   Output ~ 0
-VBAT_PAD
+BAT+
 $Comp
 L Device:R R14
